Commit message: Updated the support package to follow the new naming conventions. This package adds the 2600 12/20kg model with 165cm reach.

File: abb_irb2600_support/urdf/impl/irb2600_165_base_macro.xacro (robot description, xacro)
@@ -2,5 +2,5 @@
 <robot xmlns:xacro="http://ros.org/wiki/xacro">
   <xacro:include filename="$(find abb_resources)/urdf/common_materials.xacro"/>
-  <xacro:macro name="abb_irb2600" params="prefix">
+  <xacro:macro name="abb_irb2600_165_base" params="prefix">
     <!-- links -->
     <link name="${prefix}base_link">
@@ -8,5 +8,5 @@
         <origin xyz="0 0 0" rpy="0 0 0" />
         <geometry>
-          <mesh filename="package://abb_irb2600_support/meshes/visual/base_link.stl" />
+          <mesh filename="package://abb_irb2600_support/meshes/irb2600_165/visual/base_link.stl" />
         </geometry>
         <xacro:material_abb_orange/>
@@ -15,5 +15,5 @@
         <origin xyz="0 0 0" rpy="0 0 0" />
         <geometry>
-          <mesh filename="package://abb_irb2600_support/meshes/collision/base_link.stl" />
+          <mesh filename="package://abb_irb2600_support/meshes/irb2600_165/collision/base_link.stl" />
         </geometry>
       </collision>
@@ -23,5 +23,5 @@
         <origin xyz="0 0 0" rpy="0 0 0" />
         <geometry>
-          <mesh filename="package://abb_irb2600_support/meshes/visual/link_1.stl" />
+          <mesh filename="package://abb_irb2600_support/meshes/irb2600_165/visual/link_1.stl" />
         </geometry>
         <xacro:material_abb_orange/>
@@ -30,5 +30,5 @@
         <origin xyz="0 0 0" rpy="0 0 0" />
         <geometry>
-          <mesh filename="package://abb_irb2600_support/meshes/collision/link_1.stl" />
+          <mesh filename="package://abb_irb2600_support/meshes/irb2600_165/collision/link_1.stl" />
         </geometry>
       </collision>
@@ -38,5 +38,5 @@
         <origin xyz="0 0 0" rpy="0 0 0" />
         <geometry>
-          <mesh filename="package://abb_irb2600_support/meshes/visual/link_2.stl" />
+          <mesh filename="package://abb_irb2600_support/meshes/irb2600_165/visual/link_2.stl" />
         </geometry>
         <xacro:material_abb_orange/>
@@ -45,5 +45,5 @@
         <origin xyz="0 0 0" rpy="0 0 0" />
         <geometry>
-          <mesh filename="package://abb_irb2600_support/meshes/collision/link_2.stl" />
+          <mesh filename="package://abb_irb2600_support/meshes/irb2600_165/collision/link_2.stl" />
         </geometry>
       </collision>
@@ -53,5 +53,5 @@
         <origin xyz="0 0 0" rpy="0 0 0" />
         <geometry>
-          <mesh filename="package://abb_irb2600_support/meshes/visual/link_3.stl" />
+          <mesh filename="package://abb_irb2600_support/meshes/irb2600_165/visual/link_3.stl" />
         </geometry>
         <xacro:material_abb_orange/>
@@ -60,5 +60,5 @@
         <origin xyz="0 0 0" rpy="0 0 0" />
         <geometry>
-          <mesh filename="package://abb_irb2600_support/meshes/collision/link_3.stl" />
+          <mesh filename="package://abb_irb2600_support/meshes/irb2600_165/collision/link_3.stl" />
         </geometry>
       </collision>
@@ -68,5 +68,5 @@
         <origin xyz="0 0 0" rpy="0 0 0" />
         <geometry>
-          <mesh filename="package://abb_irb2600_support/meshes/visual/link_4.stl" />
+          <mesh filename="package://abb_irb2600_support/meshes/irb2600_165/visual/link_4.stl" />
         </geometry>
         <xacro:material_abb_orange/>
@@ -75,5 +75,5 @@
         <origin xyz="0 0 0" rpy="0 0 0" />
         <geometry>
-          <mesh filename="package://abb_irb2600_support/meshes/collision/link_4.stl" />
+          <mesh filename="package://abb_irb2600_support/meshes/irb2600_165/collision/link_4.stl" />
         </geometry>
       </collision>
@@ -83,5 +83,5 @@
         <origin xyz="0 0 0" rpy="0 0 0" />
         <geometry>
-          <mesh filename="package://abb_irb2600_support/meshes/visual/link_5.stl" />
+          <mesh filename="package://abb_irb2600_support/meshes/irb2600_165/visual/link_5.stl" />
         </geometry>
         <xacro:material_abb_orange/>
@@ -90,5 +90,5 @@
         <origin xyz="0 0 0" rpy="0 0 0" />
         <geometry>
-          <mesh filename="package://abb_irb2600_support/meshes/collision/link_5.stl" />
+          <mesh filename="package://abb_irb2600_support/meshes/irb2600_165/collision/link_5.stl" />
         </geometry>
       </collision>
@@ -98,5 +98,5 @@
         <origin xyz="0 0 0" rpy="0 0 0" />
         <geometry>
-          <mesh filename="package://abb_irb2600_support/meshes/visual/link_6.stl" />
+          <mesh filename="package://abb_irb2600_support/meshes/irb2600_165/visual/link_6.stl" />
         </geometry>
         <material name="">
@@ -107,5 +107,5 @@
         <origin xyz="0 0 0" rpy="0 0 0" />
         <geometry>
-          <mesh filename="package://abb_irb2600_support/meshes/collision/link_6.stl" />
+          <mesh filename="package://abb_irb2600_support/meshes/irb2600_165/collision/link_6.stl" />
         </geometry>
       </collision>
