Commit message: Removed the 20kg variety of 2600 in favor of a single implementation

File: abb_irb2600_support/urdf/irb2600_12_165_macro.xacro (robot description, xacro)
@@ -1,7 +1,172 @@
 <?xml version="1.0" encoding="UTF-8"?>
 <robot xmlns:xacro="http://ros.org/wiki/xacro">
-  <xacro:include filename="$(find abb_irb2600_support)/urdf/impl/irb2600_165_base_macro.xacro"/>
+  <xacro:include filename="$(find abb_resources)/urdf/common_materials.xacro"/>
   <xacro:macro name="abb_irb2600_12_165" params="prefix">
-    <xacro:abb_irb2600_165_base prefix="${prefix}"/>
+    <!-- links -->
+    <link name="${prefix}base_link">
+      <visual>
+        <origin xyz="0 0 0" rpy="0 0 0" />
+        <geometry>
+          <mesh filename="package://abb_irb2600_support/meshes/irb2600_12_165/visual/base_link.stl" />
+        </geometry>
+        <xacro:material_abb_orange/>
+      </visual>
+      <collision>
+        <origin xyz="0 0 0" rpy="0 0 0" />
+        <geometry>
+          <mesh filename="package://abb_irb2600_support/meshes/irb2600_12_165/collision/base_link.stl" />
+        </geometry>
+      </collision>
+    </link>
+    <link name="${prefix}link_1">
+      <visual>
+        <origin xyz="0 0 0" rpy="0 0 0" />
+        <geometry>
+          <mesh filename="package://abb_irb2600_support/meshes/irb2600_12_165/visual/link_1.stl" />
+        </geometry>
+        <xacro:material_abb_orange/>
+      </visual>
+      <collision>
+        <origin xyz="0 0 0" rpy="0 0 0" />
+        <geometry>
+          <mesh filename="package://abb_irb2600_support/meshes/irb2600_12_165/collision/link_1.stl" />
+        </geometry>
+      </collision>
+    </link>
+    <link name="${prefix}link_2">
+      <visual>
+        <origin xyz="0 0 0" rpy="0 0 0" />
+        <geometry>
+          <mesh filename="package://abb_irb2600_support/meshes/irb2600_12_165/visual/link_2.stl" />
+        </geometry>
+        <xacro:material_abb_orange/>
+      </visual>
+      <collision>
+        <origin xyz="0 0 0" rpy="0 0 0" />
+        <geometry>
+          <mesh filename="package://abb_irb2600_support/meshes/irb2600_12_165/collision/link_2.stl" />
+        </geometry>
+      </collision>
+    </link>
+    <link name="${prefix}link_3">
+      <visual>
+        <origin xyz="0 0 0" rpy="0 0 0" />
+        <geometry>
+          <mesh filename="package://abb_irb2600_support/meshes/irb2600_12_165/visual/link_3.stl" />
+        </geometry>
+        <xacro:material_abb_orange/>
+      </visual>
+      <collision>
+        <origin xyz="0 0 0" rpy="0 0 0" />
+        <geometry>
+          <mesh filename="package://abb_irb2600_support/meshes/irb2600_12_165/collision/link_3.stl" />
+        </geometry>
+      </collision>
+    </link>
+    <link name="${prefix}link_4">
+      <visual>
+        <origin xyz="0 0 0" rpy="0 0 0" />
+        <geometry>
+          <mesh filename="package://abb_irb2600_support/meshes/irb2600_12_165/visual/link_4.stl" />
+        </geometry>
+        <xacro:material_abb_orange/>
+      </visual>
+      <collision>
+        <origin xyz="0 0 0" rpy="0 0 0" />
+        <geometry>
+          <mesh filename="package://abb_irb2600_support/meshes/irb2600_12_165/collision/link_4.stl" />
+        </geometry>
+      </collision>
+    </link>
+    <link name="${prefix}link_5">
+      <visual>
+        <origin xyz="0 0 0" rpy="0 0 0" />
+        <geometry>
+          <mesh filename="package://abb_irb2600_support/meshes/irb2600_12_165/visual/link_5.stl" />
+        </geometry>
+        <xacro:material_abb_orange/>
+      </visual>
+      <collision>
+        <origin xyz="0 0 0" rpy="0 0 0" />
+        <geometry>
+          <mesh filename="package://abb_irb2600_support/meshes/irb2600_12_165/collision/link_5.stl" />
+        </geometry>
+      </collision>
+    </link>
+    <link name="${prefix}link_6">
+      <visual>
+        <origin xyz="0 0 0" rpy="0 0 0" />
+        <geometry>
+          <mesh filename="package://abb_irb2600_support/meshes/irb2600_12_165/visual/link_6.stl" />
+        </geometry>
+        <material name="">
+          <color rgba="0.5 0.5 0.5 1" />
+        </material>
+      </visual>
+      <collision>
+        <origin xyz="0 0 0" rpy="0 0 0" />
+        <geometry>
+          <mesh filename="package://abb_irb2600_support/meshes/irb2600_12_165/collision/link_6.stl" />
+        </geometry>
+      </collision>
+    </link>
+    <link name="${prefix}tool0" />
+    <!-- Joints -->
+    <joint name="${prefix}joint_1" type="revolute">
+      <origin xyz="0 0 0.20551" rpy="0 0 0" />
+      <parent link="${prefix}base_link" />
+      <child link="${prefix}link_1" />
+      <axis xyz="0 0 1" />
+      <limit lower="-3.14159" upper="3.14159" effort="0" velocity="3.054" />
+    </joint>
+    <joint name="${prefix}joint_2" type="revolute">
+      <origin xyz="0.14999 0 0.23949" rpy="0 0 0" />
+      <parent link="${prefix}link_1" />
+      <child link="${prefix}link_2" />
+      <axis xyz="0 1 0" />
+      <limit lower="-2.705" upper="1.658" effort="0" velocity="3.054" />
+    </joint>
+    <joint name="${prefix}joint_3" type="revolute">
+      <origin xyz="0 0 0.7" rpy="0 0 0" />
+      <parent link="${prefix}link_2" />
+      <child link="${prefix}link_3" />
+      <axis xyz="0 1 0" />
+      <limit lower="-2.705" upper="1.309" effort="0" velocity="3.054" />
+    </joint>
+    <joint name="${prefix}joint_4" type="revolute">
+      <origin xyz="0.288 0 0.115" rpy="0 0 0" />
+      <parent link="${prefix}link_3" />
+      <child link="${prefix}link_4" />
+      <axis xyz="1 0 0" />
+      <limit lower="-6.981" upper="6.981" effort="0" velocity="6.283" />
+    </joint>
+    <joint name="${prefix}joint_5" type="revolute">
+      <origin xyz="0.50733 0 0 " rpy="0 0 0" />
+      <parent link="${prefix}link_4" />
+      <child link="${prefix}link_5" />
+      <axis xyz="0 1 0" />
+      <limit lower="-2.094" upper="2.094" effort="0" velocity="6.283" />
+    </joint>
+    <joint name="${prefix}joint_6" type="revolute">
+      <origin xyz="0.056713 0 0" rpy="0 0 0" />
+      <parent link="${prefix}link_5" />
+      <child link="${prefix}link_6" />
+      <axis xyz="1 0 0" />
+      <limit lower="-6.981" upper="6.981" effort="0" velocity="8.727" />
+    </joint>
+    <joint name="${prefix}joint6-tool0" type="fixed">
+      <origin xyz="0.025958 0 0" rpy="0 1.5707963267948966 0" />
+      <parent link="${prefix}link_6" />
+      <child link="${prefix}tool0" />
+      <axis xyz="0 0 0" />
+      <limit lower="-1" upper="1" effort="0" velocity="1" />
+    </joint>
+    <!-- ROS base_link to ABB World Coordinates transform -->
+    <link name="${prefix}base" />
+    <joint name="${prefix}base_link-base" type="fixed">
+      <origin xyz="0 0 0" rpy="0 0 0" />
+      <parent link="${prefix}base_link" />
+      <child link="${prefix}base" />
+    </joint>
   </xacro:macro>
 </robot>

Commit message: Minor changes. To be squashed.

File: abb_irb2600_support/urdf/irb2600_12_165_macro.xacro (robot description, xacro)
@@ -159,6 +159,4 @@
       <parent link="${prefix}link_6" />
       <child link="${prefix}tool0" />
-      <axis xyz="0 0 0" />
-      <limit lower="-1" upper="1" effort="0" velocity="1" />
     </joint>
     <!-- ROS base_link to ABB World Coordinates transform -->
