Commit message: Testing

File: abb_irb4600_support/urdf/irb4600_60_205_macro.xacro (robot description, xacro)
@@ -118,5 +118,6 @@
       <parent link="${prefix}link_2"/>
       <child link="${prefix}link_3"/>
-      <limit effort="0" lower="-3.141" upper="1.308" velocity="3.054"/>
+      <!-- Nominally negative pi for lower limit -->
+      <limit effort="0" lower="-2.5" upper="1.2" velocity="3.054"/>
     </joint>
     <joint type="revolute" name="${prefix}joint_4">
